File: leg/pcbs/as5048a_diff_spi_breakout/as5048a_diff_spi_breakout.kicad_sch (KiCad schematic)
At the start: 8 parts, among them J1 Conn_01x02, J2 8P8C, U1 SN65LVDT14, U2 AS5048A

Commit message: folder restructure
Parts:
- J1: Manufacturer Number (none) -> 0436500212
- J2: Manufacturer Number (none) -> RJSSE508001T
Other:
- note added: "AS5048A Diff SPI Breakout"
Changed lines of the file:
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@@
     (stroke (width 0) (type default) (color 0 0 0 0))
+  )
+  (text "AS5048A Diff SPI Breakout" (at 186.69 190.5 0)
+    (effects (font (size 1.27 1.27)) (justify left bottom))
   )
   (text "Pwr Connector" (at 29.21 21.59 0)
@@
       (effects (font (size 1.27 1.27)) hide)
     )
+    (property "Manufacturer Number" "RJSSE508001T" (id 4) (at 93.98 92.71 0)
+      (effects (font (size 1.27 1.27)) hide)
+    )
     (pin "1")
     (pin "2")
@@
       (effects (font (size 1.27 1.27)) hide)
     )
+    (property "Manufacturer Number" "0436500212" (id 4) (at 22.86 35.56 0)
+      (effects (font (size 1.27 1.27)) hide)
+    )
