File: leg/pcbs/odrive_diff_spi_breakout/odrive_diff_spi_breakout.kicad_sch (KiCad schematic)
At the start: 17 parts, among them J1 Conn_01x02, J2 Conn_01x02, J3 Conn_01x20, J4 8P8C, J5 8P8C, U1 74CBTLV1G125, U2 74CBTLV1G125, U3 SN65LVDT41, U4 SN65LVDT41

Commit message: folder restructure
Parts:
- J1, J2: Manufacturer Number (none) -> 0436500215
- U1, U2: Manufacturer Number (none) -> 74CBTLV1G125DBVRQ1
Other:
- note added: "Note 1: Bus Switches are placed on MISO lines (enabled when CS = 0) to avoid contention. Normal devices put MISO lines in high impedance state when not in communication."
- note added: "ODrive Dual Diff SPI Breakout"
- note added: "See Note 1."
Changed lines of the file:
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@@
     (stroke (width 0) (type default) (color 0 0 0 0))
   )
+  (text "ODrive Dual Diff SPI Breakout" (at 186.69 190.5 0)
+    (effects (font (size 1.27 1.27)) (justify left bottom))
+  )
   (text "GPIO8" (at 74.93 104.14 0)
     (effects (font (size 1.27 1.27)) (justify left bottom))
@@
     (effects (font (size 1.27 1.27)) (justify left bottom))
   )
+  (text "See Note 1." (at 106.68 85.09 0)
+    (effects (font (size 1.27 1.27)) (justify left bottom))
+  )
   (text "GPIO6" (at 74.93 99.06 0)
     (effects (font (size 1.27 1.27)) (justify left bottom))
@@
   )
   (text "GPIO2" (at 74.93 88.9 0)
+    (effects (font (size 1.27 1.27)) (justify left bottom))
+  )
+  (text "See Note 1." (at 106.68 143.51 0)
+    (effects (font (size 1.27 1.27)) (justify left bottom))
+  )
+  (text "Note 1: Bus Switches are placed on MISO lines\n(enabled when CS = 0) to avoid contention.\nNormal devices put MISO lines in high impedance state\nwhen not in communication."
+    (at 119.38 194.31 0)
     (effects (font (size 1.27 1.27)) (justify left bottom))
   )
@@
       (effects (font (size 1.27 1.27)) hide)
     )
+    (property "Manufacturer Number" "74CBTLV1G125DBVRQ1" (id 4) (at 120.65 90.17 0)
+      (effects (font (size 1.27 1.27)) hide)
+    )
     (pin "1")
     (pin "2")
@@
       (effects (font (size 1.27 1.27)) hide)
     )
+    (property "Manufacturer Number" "74CBTLV1G125DBVRQ1" (id 4) (at 120.65 148.59 0)
+      (effects (font (size 1.27 1.27)) hide)
+    )
     (pin "1")
     (pin "2")
@@
     )
     (property "Datasheet" "~" (id 3) (at 62.23 181.61 0)
+      (effects (font (size 1.27 1.27)) hide)
+    )
+    (property "Manufacturer Number" "0436500215" (id 4) (at 62.23 181.61 0)
       (effects (font (size 1.27 1.27)) hide)
     )
@@
       (effects (font (size 1.27 1.27)) hide)
     )
+    (property "Manufacturer Number" "0436500215" (id 4) (at 29.21 181.61 0)
+      (effects (font (size 1.27 1.27)) hide)
+    )
